File: KiCad/zwischenkreis/zwischenkreis.kicad_sch (KiCad schematic)
At the start: 39 parts, among them J1 Conn_01x01_Pin, J2 Conn_01x01_Pin, J3 Conn_01x01_Pin, J4 Conn_01x01_Pin, J5 Conn_01x01_Pin, J6 Conn_01x01_Pin, Q1 SS8550, Q10 IRF540N, Q12 2N3904, Q13 2N3904, Q14 SS8050, Q15 2N3904, Q16 2N3904, Q17 SS8050, Q2 SS8550, Q9 IRF540N

Commit message: Test Software aufgesetzt
Parts:
- removed C3, C4: 300n/50V, Capacitor_THT:C_Disc_D5.0mm_W2.5mm_P5.00mm, symbol Device:C
- removed C5, C6: 22p/50V, Capacitor_THT:C_Disc_D5.0mm_W2.5mm_P5.00mm, symbol Device:C
- removed D3, D4, D5: 1N4007, Diode_THT:D_DO-41_SOD81_P7.62mm_Horizontal, symbol Device:D
- removed H1, H2, H3, H4: MountingHole, MountingHole:MountingHole_2.2mm_M2_ISO14580_Pad, symbol Mechanical:MountingHole
- removed J1, J2, J3, J4, J5, J6: Conn_01x01_Pin, Connector_PinHeader_2.54mm:PinHeader_1x01_P2.54mm_Vertical, symbol Connector:Conn_01x01_Pin
- removed Q1, Q2: SS8550, Package_TO_SOT_THT:TO-92L_Inline_Wide, symbol Transistor_BJT:2N3905
- removed Q10, Q9: IRF540N, Package_TO_SOT_THT:TO-220-3_Horizontal_TabUp, symbol Transistor_FET:IRF540N
- removed Q12, Q13, Q15, Q16: 2N3904, Package_TO_SOT_THT:TO-92L_Inline_Wide, symbol Transistor_BJT:2N3904
- removed Q14, Q17: SS8050, Package_TO_SOT_THT:TO-92L_Inline_Wide, symbol Transistor_BJT:2N3904
- removed R1, R2, R3, R4: 5k1, Resistor_THT:R_Axial_DIN0204_L3.6mm_D1.6mm_P7.62mm_Horizontal, symbol Device:R
- removed R10, R9: 10R, Resistor_THT:R_Axial_DIN0204_L3.6mm_D1.6mm_P7.62mm_Horizontal, symbol Device:R
- removed R11, R12: 100k, Resistor_THT:R_Axial_DIN0204_L3.6mm_D1.6mm_P7.62mm_Horizontal, symbol Device:R
- removed R5, R6, R7, R8: 10k, Resistor_THT:R_Axial_DIN0204_L3.6mm_D1.6mm_P7.62mm_Horizontal, symbol Device:R
- added C1: 470u, symbol Device:C_Polarized
- added C11: 300n/50V, Capacitor_THT:C_Disc_D5.0mm_W2.5mm_P5.00mm, symbol Device:C
- added J13, J14, J15, J16, J17, J18: Conn_01x01_Pin, Connector_PinHeader_2.54mm:PinHeader_1x01_P2.54mm_Vertical, symbol Connector:Conn_01x01_Pin
- added R25: 10k, Resistor_THT:R_Axial_DIN0204_L3.6mm_D1.6mm_P7.62mm_Horizontal, symbol Device:R
Connections:
- net GND: now also C1.2, C11.2, J14.1 (Pin_1), J17.1 (Pin_1), J18.1 (Pin_1), R25.2
- new net VDC: C1.1, C11.1, J13.1 (Pin_1), J15.1 (Pin_1), J16.1 (Pin_1), R25.1
Other:
- note added: "GND h-bridge 1"
- note added: "GND h-bridge 2"
- note added: "VDC"
- note added: "VDC h-bridge 1"
- note added: "VDC h-bridge 2"
- note removed: "+18V"
- note removed: "OUT"
- note removed: "PWM_HIGH"
- note removed: "PWM_LOW"
- note removed: "µC GND"
- title: halbbruecke -> zwischenkreis
